Commit message: gazebo running

File: asclepius/urdf/asclepius.urdf.xacro (robot description, xacro)
@@ -2,7 +2,6 @@
 <robot name="asclepius" xmlns:xacro="http://ros.org/wiki/xacro">
   <xacro:include filename="$(find asclepius)/urdf/asclepius.xacro" />
-  <!-- <xacro:include filename="$(find dynamixel_arm)/urdf/acps_bot.ros2_control_gazebo.xacro" /> -->
-  <!-- <link name="world"/> -->
-  <xacro:asclepius/>
-  <!-- <xacro:acps_bot_ros2_control_gazebo name="acps_bot_ros2_control_gazebo" /> -->
+  <xacro:include filename="$(find asclepius)/urdf/ros2_control_gazebo.xacro" />
+  <xacro:robot/>
+  <xacro:GZSystem/>
 </robot>

File: asclepius/urdf/asclepius.xacro (robot description, xacro)
@@ -1,5 +1,5 @@
 <?xml version="1.0"?>
 <robot xmlns:xacro="http://www.ros.org/wiki/xacro">
-<xacro:macro name="asclepius">
+<xacro:macro name="robot">
   <link name="world"/>
   <joint name="origin_to_joint1" type="fixed">
@@ -30,5 +30,5 @@
       <geometry>
         <mesh
-          filename="package://asclepius/meshes/base_link.STL" />
+          filename="file://$(find asclepius)/meshes/base_link.STL" />
       </geometry>
       <material
@@ -44,5 +44,5 @@
       <geometry>
         <mesh
-          filename="package://asclepius/meshes/base_link.STL" />
+          filename="file://$(find asclepius)/meshes/base_link.STL" />
       </geometry>
     </collision>
@@ -70,5 +70,5 @@
       <geometry>
         <mesh
-          filename="package://asclepius/meshes/link1.STL" />
+          filename="file://$(find asclepius)/meshes/link1.STL" />
       </geometry>
       <material
@@ -84,5 +84,5 @@
       <geometry>
         <mesh
-          filename="package://asclepius/meshes/link1.STL" />
+          filename="file://$(find asclepius)/meshes/link1.STL" />
       </geometry>
     </collision>
@@ -123,5 +123,5 @@
       <geometry>
         <mesh
-          filename="package://asclepius/meshes/link2.STL" />
+          filename="file://$(find asclepius)/meshes/link2.STL" />
       </geometry>
       <material
@@ -137,5 +137,5 @@
       <geometry>
         <mesh
-          filename="package://asclepius/meshes/link2.STL" />
+          filename="file://$(find asclepius)/meshes/link2.STL" />
       </geometry>
     </collision>
@@ -176,5 +176,5 @@
       <geometry>
         <mesh
-          filename="package://asclepius/meshes/link3.STL" />
+          filename="file://$(find asclepius)/meshes/link3.STL" />
       </geometry>
       <material
@@ -190,5 +190,5 @@
       <geometry>
         <mesh
-          filename="package://asclepius/meshes/link3.STL" />
+          filename="file://$(find asclepius)/meshes/link3.STL" />
       </geometry>
     </collision>
@@ -229,5 +229,5 @@
       <geometry>
         <mesh
-          filename="package://asclepius/meshes/link4.STL" />
+          filename="file://$(find asclepius)/meshes/link4.STL" />
       </geometry>
       <material
@@ -243,5 +243,5 @@
       <geometry>
         <mesh
-          filename="package://asclepius/meshes/link4.STL" />
+          filename="file://$(find asclepius)/meshes/link4.STL" />
       </geometry>
     </collision>
@@ -282,5 +282,5 @@
       <geometry>
         <mesh
-          filename="package://asclepius/meshes/link5.STL" />
+          filename="file://$(find asclepius)/meshes/link5.STL" />
       </geometry>
       <material
@@ -296,5 +296,5 @@
       <geometry>
         <mesh
-          filename="package://asclepius/meshes/link5.STL" />
+          filename="file://$(find asclepius)/meshes/link5.STL" />
       </geometry>
     </collision>
@@ -335,5 +335,5 @@
       <geometry>
         <mesh
-          filename="package://asclepius/meshes/link6.STL" />
+          filename="file://$(find asclepius)/meshes/link6.STL" />
       </geometry>
       <material
@@ -349,5 +349,5 @@
       <geometry>
         <mesh
-          filename="package://asclepius/meshes/link6.STL" />
+          filename="file://$(find asclepius)/meshes/link6.STL" />
       </geometry>
     </collision>
@@ -388,5 +388,5 @@
       <geometry>
         <mesh
-          filename="package://asclepius/meshes/link7.STL" />
+          filename="file://$(find asclepius)/meshes/link7.STL" />
       </geometry>
       <material
@@ -402,5 +402,5 @@
       <geometry>
         <mesh
-          filename="package://asclepius/meshes/link7.STL" />
+          filename="file://$(find asclepius)/meshes/link7.STL" />
       </geometry>
     </collision>

File: dynamixel_arm/urdf/acps_bot.xacro (robot description, xacro)
@@ -25,19 +25,19 @@
         <geometry>
             <mesh
-            filename="package://dynamixel_arm/meshes/base_link.STL" />
-        </geometry>
-        <material
-            name="">
-            <color
-            rgba="0.79216 0.81961 0.93333 1" />
-        </material>
-        </visual>
-        <collision>
-        <origin
-            xyz="0 0 0"
-            rpy="0 0 0" />
-        <geometry>
-            <mesh
-            filename="package://dynamixel_arm/meshes/base_link.STL" />
+            filename="file://$(find dynamixel_arm)/meshes/base_link.STL" />
+        </geometry>
+        <material
+            name="">
+            <color
+            rgba="0.79216 0.81961 0.93333 1" />
+        </material>
+        </visual>
+        <collision>
+        <origin
+            xyz="0 0 0"
+            rpy="0 0 0" />
+        <geometry>
+            <mesh
+            filename="file://$(find dynamixel_arm)/meshes/base_link.STL" />
         </geometry>
         </collision>
@@ -65,19 +65,19 @@
         <geometry>
             <mesh
-            filename="package://dynamixel_arm/meshes/link1.STL" />
-        </geometry>
-        <material
-            name="">
-            <color
-            rgba="0.79216 0.81961 0.93333 1" />
-        </material>
-        </visual>
-        <collision>
-        <origin
-            xyz="0 0 0"
-            rpy="0 0 0" />
-        <geometry>
-            <mesh
-            filename="package://dynamixel_arm/meshes/link1.STL" />
+            filename="file://$(find dynamixel_arm)/meshes/link1.STL" />
+        </geometry>
+        <material
+            name="">
+            <color
+            rgba="0.79216 0.81961 0.93333 1" />
+        </material>
+        </visual>
+        <collision>
+        <origin
+            xyz="0 0 0"
+            rpy="0 0 0" />
+        <geometry>
+            <mesh
+            filename="file://$(find dynamixel_arm)/meshes/link1.STL" />
         </geometry>
         </collision>
@@ -105,19 +105,19 @@
         <geometry>
             <mesh
-            filename="package://dynamixel_arm/meshes/link2.STL" />
-        </geometry>
-        <material
-            name="">
-            <color
-            rgba="0.79216 0.81961 0.93333 1" />
-        </material>
-        </visual>
-        <collision>
-        <origin
-            xyz="0 0 0"
-            rpy="0 0 0" />
-        <geometry>
-            <mesh
-            filename="package://dynamixel_arm/meshes/link2.STL" />
+            filename="file://$(find dynamixel_arm)/meshes/link2.STL" />
+        </geometry>
+        <material
+            name="">
+            <color
+            rgba="0.79216 0.81961 0.93333 1" />
+        </material>
+        </visual>
+        <collision>
+        <origin
+            xyz="0 0 0"
+            rpy="0 0 0" />
+        <geometry>
+            <mesh
+            filename="file://$(find dynamixel_arm)/meshes/link2.STL" />
         </geometry>
         </collision>
@@ -145,19 +145,19 @@
         <geometry>
             <mesh
-            filename="package://dynamixel_arm/meshes/link3.STL" />
-        </geometry>
-        <material
-            name="">
-            <color
-            rgba="0.79216 0.81961 0.93333 1" />
-        </material>
-        </visual>
-        <collision>
-        <origin
-            xyz="0 0 0"
-            rpy="0 0 0" />
-        <geometry>
-            <mesh
-            filename="package://dynamixel_arm/meshes/link3.STL" />
+            filename="file://$(find dynamixel_arm)/meshes/link3.STL" />
+        </geometry>
+        <material
+            name="">
+            <color
+            rgba="0.79216 0.81961 0.93333 1" />
+        </material>
+        </visual>
+        <collision>
+        <origin
+            xyz="0 0 0"
+            rpy="0 0 0" />
+        <geometry>
+            <mesh
+            filename="file://$(find dynamixel_arm)/meshes/link3.STL" />
         </geometry>
         </collision>
@@ -185,19 +185,19 @@
         <geometry>
             <mesh
-            filename="package://dynamixel_arm/meshes/link4.STL" />
-        </geometry>
-        <material
-            name="">
-            <color
-            rgba="0.79216 0.81961 0.93333 1" />
-        </material>
-        </visual>
-        <collision>
-        <origin
-            xyz="0 0 0"
-            rpy="0 0 0" />
-        <geometry>
-            <mesh
-            filename="package://dynamixel_arm/meshes/link4.STL" />
+            filename="file://$(find dynamixel_arm)/meshes/link4.STL" />
+        </geometry>
+        <material
+            name="">
+            <color
+            rgba="0.79216 0.81961 0.93333 1" />
+        </material>
+        </visual>
+        <collision>
+        <origin
+            xyz="0 0 0"
+            rpy="0 0 0" />
+        <geometry>
+            <mesh
+            filename="file://$(find dynamixel_arm)/meshes/link4.STL" />
         </geometry>
         </collision>
