Commit message: rough kinematics

File: asclepius/description/asclepius.urdf.xacro (robot description, xacro)
@@ -1,9 +1,7 @@
 <?xml version="1.0"?>
 <robot name="asclepius" xmlns:xacro="http://ros.org/wiki/xacro">
-  <xacro:include filename="$(find asclepius)/description/asclepius.xacro" />
-  <!-- <xacro:include filename="$(find asclepius)/description/ros2_control_gazebo.xacro" /> -->
-  <xacro:include filename="$(find asclepius)/description/hardware_control.xacro" />
-  <xacro:robot/>
-  <xacro:hardware_control/>
-  <!-- <xacro:GZSystem/> -->
+  <!-- <xacro:include filename="$(find asclepius)/description/asclepius.xacro" /> -->
+  <!-- <xacro:include filename="$(find asclepius)/description/hardware_control.xacro" /> -->
+  <!-- <xacro:robot/> -->
+  <!-- <xacro:hardware_control/> -->
 </robot>

File: asclepius/description/asclepius.xacro (robot description, xacro)
@@ -1,4 +1,5 @@
 <?xml version="1.0"?>
 <robot xmlns:xacro="http://www.ros.org/wiki/xacro">
+<xacro:include filename="$(find asclepius)/description/util.xacro" />
 <xacro:macro name="robot">
   <link name="world"/>
@@ -33,8 +34,5 @@
       </geometry>
       <material
-        name="">
-        <color
-          rgba="0.792156862745098 0.819607843137255 0.933333333333333 1" />
-      </material>
+        name="red"/>
     </visual>
     <collision>
@@ -72,9 +70,5 @@
           filename="file://$(find asclepius)/meshes/link1.STL" />
       </geometry>
-      <material
-        name="">
-        <color
-          rgba="0.79216 0.81961 0.93333 1" />
-      </material>
+      <material name="blue"/>
     </visual>
     <collision>
@@ -126,8 +120,5 @@
       </geometry>
       <material
-        name="">
-        <color
-          rgba="0.79216 0.81961 0.93333 1" />
-      </material>
+        name="magenta"/>
     </visual>
     <collision>
@@ -179,8 +170,5 @@
       </geometry>
       <material
-        name="">
-        <color
-          rgba="0.792156862745098 0.819607843137255 0.933333333333333 1" />
-      </material>
+        name="green"/>
     </visual>
     <collision>
@@ -232,8 +220,5 @@
       </geometry>
       <material
-        name="">
-        <color
-          rgba="0.25098 0.25098 0.25098 1" />
-      </material>
+        name="cyan"/>
     </visual>
     <collision>
@@ -285,8 +270,5 @@
       </geometry>
       <material
-        name="">
-        <color
-          rgba="0.75294 0.75294 0.75294 1" />
-      </material>
+        name="magenta"/>
     </visual>
     <collision>
@@ -338,8 +320,5 @@
       </geometry>
       <material
-        name="">
-        <color
-          rgba="0.59216 0.50196 0.50196 1" />
-      </material>
+        name="red"/>
     </visual>
     <collision>
@@ -391,8 +370,5 @@
       </geometry>
       <material
-        name="">
-        <color
-          rgba="0.59216 0.50196 0.50196 1" />
-      </material>
+        name="blue"/>
     </visual>
     <collision>

File: asclepius/description/hardware_control.xacro (robot description, xacro)
@@ -1,3 +1,3 @@
-<?xml version="1.0"?>
+<!-- <?xml version="1.0"?>
 <robot xmlns:xacro="http://www.ros.org/wiki/xacro">
   <xacro:macro name="hardware_control">
@@ -47,3 +47,3 @@
     </ros2_control>
   </xacro:macro>
-</robot>
+</robot> -->

File: asclepius/description/ros2_control_gazebo.xacro (robot description, xacro)
@@ -48,11 +48,11 @@
         <!-- <state_interface name="effort"/> -->
       </joint>
-      <joint name="joint7">
-        <command_interface name="position"/>
+      <!-- <joint name="joint7"> -->
+        <!-- <command_interface name="position"/> -->
         <!-- <command_interface name="velocity"/> -->
-        <state_interface name="position"/>
-        <state_interface name="velocity"/>
+        <!-- <state_interface name="position"/> -->
+        <!-- <state_interface n/ame="velocity"/> -->
         <!-- <state_interface name="effort"/> -->
-      </joint>
+      <!-- </joint> -->
     </ros2_control>
   <gazebo>

Commit message: ahhhh

File: asclepius/description/asclepius.urdf.xacro (robot description, xacro)
@@ -1,7 +1,8 @@
 <?xml version="1.0"?>
-<robot name="asclepius" xmlns:xacro="http://ros.org/wiki/xacro">
-  <!-- <xacro:include filename="$(find asclepius)/description/asclepius.xacro" /> -->
-  <!-- <xacro:include filename="$(find asclepius)/description/hardware_control.xacro" /> -->
-  <!-- <xacro:robot/> -->
-  <!-- <xacro:hardware_control/> -->
+<robot name="asclepius"
+  xmlns:xacro="http://ros.org/wiki/xacro">
+  <xacro:include filename="$(find asclepius)/description/asclepius.xacro" />
+  <xacro:include filename="$(find asclepius)/description/hardware_control.xacro" />
+  <xacro:robot/>
+  <xacro:hardware_control/>
 </robot>

File: asclepius/description/hardware_control.xacro (robot description, xacro)
@@ -1,7 +1,43 @@
-<!-- <?xml version="1.0"?>
+<?xml version="1.0"?>
 <robot xmlns:xacro="http://www.ros.org/wiki/xacro">
   <xacro:macro name="hardware_control">
+    <ros2_control name="fake_hardware_control" type="system">
+      <hardware>
+        <plugin>dynamixel_hardware/DynamixelHardware</plugin>
+        <param name="usb_port">/dev/ttyUSB1</param>
+        <param name="baud_rate">1000000</param>
+        <param name="use_dummy">true</param>
+      </hardware>
+      <!-- Twist rotattion -->
+      <joint name="joint1">
+        <param name="id">1</param>
+        <command_interface name="position"/>
+        <!-- <command_interface name="velocity"/> -->
+        <state_interface name="position"/>
+        <!-- <state_interface name="velocity"/> -->
+        <!-- <state_interface name="effort"/> -->
+      </joint>
+      <!-- Side to side -->
+      <joint name="joint2">
+        <param name="id">2</param>
+        <command_interface name="position"/>
+        <!-- <command_interface name="velocity"/> -->
+        <state_interface name="position"/>
+        <!-- <state_interface name="velocity"/> -->
+        <!-- <state_interface name="effort"/> -->
+      </joint>
+      <!-- Left Claw -->
+      <joint name="joint3">
+        <param name="id">3</param>
+        <command_interface name="position"/>
+        <!-- <command_interface name="velocity"/> -->
+        <state_interface name="position"/>
+        <!-- <state_interface name="velocity"/> -->
+        <!-- <state_interface name="effort"/> -->
+      </joint>
+    </ros2_control>
     <ros2_control name="hardware_control" type="system">
       <hardware>
+        <!-- <plugin>endeffector_hardware/EndeffectorHardware</plugin> -->
         <plugin>dynamixel_hardware/DynamixelHardware</plugin>
         <param name="usb_port">/dev/ttyUSB0</param>
@@ -9,12 +45,12 @@
         <!-- <param name="use_dummy">true</param> -->
       </hardware>
-        <!-- Twist rotattion -->
+      <!-- Twist rotattion -->
       <joint name="joint4">
         <param name="id">7</param>
         <command_interface name="position"/>
-        <command_interface name="velocity"/>
+        <!-- <command_interface name="velocity"/> -->
         <state_interface name="position"/>
-        <state_interface name="velocity"/>
-        <state_interface name="effort"/>
+        <!-- <state_interface name="velocity"/> -->
+        <!-- <state_interface name="effort"/> -->
       </joint>
       <!-- Side to side -->
@@ -22,17 +58,17 @@
         <param name="id">9</param>
         <command_interface name="position"/>
-        <command_interface name="velocity"/>
+        <!-- <command_interface name="velocity"/> -->
         <state_interface name="position"/>
-        <state_interface name="velocity"/>
-        <state_interface name="effort"/>
+        <!-- <state_interface name="velocity"/> -->
+        <!-- <state_interface name="effort"/> -->
       </joint>
-    <!-- Left Claw -->
-    <joint name="joint6">
+      <!-- Left Claw -->
+      <joint name="joint6">
         <param name="id">11</param>
         <command_interface name="position"/>
-        <command_interface name="velocity"/>
+        <!-- <command_interface name="velocity"/> -->
         <state_interface name="position"/>
-        <state_interface name="velocity"/>
-        <state_interface name="effort"/>
+        <!-- <state_interface name="velocity"/> -->
+        <!-- <state_interface name="effort"/> -->
       </joint>
       <!-- Right Claw -->
@@ -40,10 +76,10 @@
         <param name="id">10</param>
         <command_interface name="position"/>
-        <command_interface name="velocity"/>
+        <!-- <command_interface name="velocity"/> -->
         <state_interface name="position"/>
-        <state_interface name="velocity"/>
-        <state_interface name="effort"/>
+        <!-- <state_interface name="velocity"/> -->
+        <!-- <state_interface name="effort"/> -->
       </joint>
     </ros2_control>
   </xacro:macro>
-</robot> -->
+</robot>
